File: testing-schematics/Logic testing/Logic testing.kicad_sch (KiCad schematic)
At the start: 43 parts, among them IC1 ESP32-C6-WROOM-1U-N8, J1 External Box, J2 Aux Wire, J3 Conn_01x04, J4 Lame Tab, J5 Test Output, K1 G6K-2, K2 G6K-2, K3 G6K-2, K4 G6K-2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

Commit message: Worked on connectors, PCB layout, created footprints, component CAD, journal
Parts:
- added H1, H2, H3, H4: MountingHole, MountingHole:MountingHole_3.2mm_M3_ISO7380_Pad_TopBottom, symbol Mechanical:MountingHole
- added H5, H6, H7, H8: MountingHole, symbol Mechanical:MountingHole
- J1, J2, J5: footprint (none) -> Custom:Fencing Plug
Other:
- note added: "Board Mounting"
- note added: "Screen Mounting"

Commit message: Work from 14th
Parts:
- added J6: Small Pin, Connector_Wire:SolderWire-0.5sqmm_1x01_D0.9mm_OD2.1mm, symbol Connector_Generic:Conn_01x01
- SW3: footprint Button_Switch_THT:SW_PUSH-12mm -> Button_Switch_THT:SW_PUSH_6mm_H13mm
Connections:
- net B2: now also J6.1 (Pin_1)
Changed lines of the file:
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@@
 		)
 	)
+	(label "3.3V"
+		(at 57.15 93.98 0)
+		(effects
+			(font
+				(size 1.27 1.27)
+			)
+			(justify left bottom)
+		)
+	)
 	(global_label "BTN USE"
 		(shape input)
@@
 		)
 	)
+	(global_label "B2"
+		(shape input)
+		(at 93.98 78.74 0)
+		(fields_autoplaced yes)
+		(effects
+			(font
+				(size 1.27 1.27)
+			)
+			(justify left)
+		)
+		(property "Intersheetrefs" "${INTERSHEET_REFS}"
+			(at 99.4447 78.74 0)
+			(effects
+				(font
+					(size 1.27 1.27)
+				)
+				(justify left)
+				(hide yes)
+			)
+		)
+	)
 	(global_label "USB_D-"
 		(shape input)
@@
 	)
 	(symbol
+		(lib_id "Connector_Generic:Conn_01x01")
+		(at 88.9 78.74 0)
+		(mirror y)
+		(unit 1)
+		(exclude_from_sim no)
+		(in_bom yes)
+		(on_board yes)
+		(dnp no)
+		(property "Reference" "J6"
+			(at 81.788 77.724 0)
+			(effects
+				(font
+					(size 1.27 1.27)
+				)
+			)
+		)
+		(property "Value" "Small Pin"
+			(at 82.042 79.756 0)
+			(effects
+				(font
+					(size 1.27 1.27)
+				)
+			)
+		)
+		(property "Footprint" "Connector_Wire:SolderWire-0.5sqmm_1x01_D0.9mm_OD2.1mm"
+			(at 88.9 78.74 0)
+			(effects
+				(font
+					(size 1.27 1.27)
+				)
+				(hide yes)
+			)
+		)
+		(property "Datasheet" "~"
+			(at 88.9 78.74 0)
+			(effects
+				(font
+					(size 1.27 1.27)
+				)
+				(hide yes)
+			)
+		)
+		(property "Description" "Generic connector, single row, 01x01, script generated (kicad-library-utils/schlib/autogen/connector/)"
+			(at 88.9 78.74 0)
+			(effects
+				(font
+					(size 1.27 1.27)
+				)
+				(hide yes)
+			)
+		)
+		(property "Description_1" ""
+			(at 88.9 78.74 0)
+			(effects
+				(font
+					(size 1.27 1.27)
+				)
+			)
+		)
+		(property "MF" ""
+			(at 88.9 78.74 0)
+			(effects
+				(font
+					(size 1.27 1.27)
+				)
+			)
+		)
+		(property "MP" ""
+			(at 88.9 78.74 0)
+			(effects
+				(font
+					(size 1.27 1.27)
+				)
+			)
+		)
+		(property "PACKAGE" ""
+			(at 88.9 78.74 0)
+			(effects
+				(font
+					(size 1.27 1.27)
+				)
+			)
+		)
+		(property "Package" ""
+			(at 88.9 78.74 0)
+			(effects
+				(font
+					(size 1.27 1.27)
+				)
+			)
+		)
+		(pin "1"
+		)
+		(instances
+			(project "Logic testing"
+				(path "/084a3cde-ed27-4296-b8ef-5d12812311e6"
+					(reference "J6")
+					(unit 1)
+				)
+			)
+		)
+	)
+	(symbol
 		(lib_id "Device:R")
 		(at 176.53 74.93 0)
@@
 			)
 		)
-		(property "Footprint" "Button_Switch_THT:SW_PUSH-12mm"
+		(property "Footprint" "Button_Switch_THT:SW_PUSH_6mm_H13mm"
 			(at 96.52 86.36 0)
 			(effects

Commit message: Finished PCB; Updated USB-C connector; Stated on CAD
Parts:
- H5, H6, H7, H8: footprint (none) -> MountingHole:MountingHole_2.2mm_M2_DIN965_Pad_TopBottom
- P1: footprint Connector_USB:USB_C_Receptacle_GCT_USB4105-xx-A_16P_TopMnt_Horizontal -> Connector_USB:USB_C_Receptacle_GCT_USB4085
Changed lines of the file:
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@@
 			)
 		)
-		(property "Footprint" ""
+		(property "Footprint" "MountingHole:MountingHole_2.2mm_M2_DIN965_Pad_TopBottom"
 			(at 147.32 111.76 0)
 			(effects
@@
 			)
 		)
-		(property "Footprint" ""
+		(property "Footprint" "MountingHole:MountingHole_2.2mm_M2_DIN965_Pad_TopBottom"
 			(at 147.32 127 0)
 			(effects
@@
 			)
 		)
-		(property "Footprint" ""
+		(property "Footprint" "MountingHole:MountingHole_2.2mm_M2_DIN965_Pad_TopBottom"
 			(at 147.32 116.84 0)
 			(effects
@@
 			)
 		)
-		(property "Footprint" "Connector_USB:USB_C_Receptacle_GCT_USB4105-xx-A_16P_TopMnt_Horizontal"
+		(property "Footprint" "Connector_USB:USB_C_Receptacle_GCT_USB4085"
 			(at 29.21 129.54 0)
 			(effects
@@
 			)
 		)
-		(property "Footprint" ""
+		(property "Footprint" "MountingHole:MountingHole_2.2mm_M2_DIN965_Pad_TopBottom"
 			(at 147.32 121.92 0)
 			(effects

Commit message: Worked on  issues
Parts:
- added D5: 1N4148, Diode_SMD:D_SOD-123, symbol Diode:1N4148
- added K6: G6K-2, Relay_SMD:Relay_DPDT_Omron_G6K-2F, symbol Relay:G6K-2
- added Q5: BC547, Package_TO_SOT_THT:TO-92_Inline, symbol Transistor_BJT:BC547
- added R16, R17: 10k, Custom:R_1206_3216Metric_Pad1.30x1.75mm_HandSolder_Text, symbol Device:R
- added R8: 510, Custom:R_1206_3216Metric_Pad1.30x1.75mm_HandSolder_Text, symbol Device:R
- C3: footprint Capacitor_SMD:C_0603_1608Metric_Pad1.08x0.95mm_HandSolder -> Capacitor_SMD:C_0805_2012Metric_Pad1.18x1.45mm_HandSolder
- D1, D2, D3, D4: footprint Diode_THT:D_DO-35_SOD27_P7.62mm_Horizontal -> Diode_SMD:D_SOD-123
- R1, R11, R12, R13, R14, R15, R2, R3, R4, R5, R6, R7, R9: footprint Resistor_SMD:R_1206_3216Metric_Pad1.30x1.75mm_HandSolder -> Custom:R_1206_3216Metric_Pad1.30x1.75mm_HandSolder_Text
Connections:
- net +5V: now also D5.1 (K), K6.1
- net GND: now also IC1.10 (IO8), IC1.15 (IO9), Q5.3 (E), R16.1, R17.1
- net SG1: now also K6.4; no longer K4.4
- net WT1: now also R17.2; no longer IC1.10 (IO8)
- net WT3: now also R16.2; no longer IC1.15 (IO9)
- new net: Q5.2 (B), R8.2
- new net: D5.2 (A), K6.8, Q5.1 (C)
- new net: K4.4, K6.3
- new net REL5: R8.1
- no-connect marks 16 -> 20
Other:
- moved on the sheet: D2, D3, D4, J4, Q2, Q3, Q4, R2, R3, R6

Commit message: Worked on PCB; worked on Code; Worked on journal
Connections:
- net REL5: now also IC1.19 (IO21)
- no-connect marks 20 -> 19
Changed lines of the file:
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@@
-	)
-	(no_connect
-		(at 25.4 82.55)
 	)
 	(no_connect
@@
 				(hide yes)
 			)
+		)
+	)
+	(global_label "REL5"
+		(shape input)
+		(at 25.4 82.55 180)
+		(fields_autoplaced yes)
+		(effects
+			(font
+				(size 1.27 1.27)
+			)
+			(justify right)
+		)
+		(property "Intersheetrefs" "${INTERSHEET_REFS}"
+			(at 17.7582 82.55 0)
+			(effects
+				(font
+					(size 1.27 1.27)
+				)
+				(justify right)
+				(hide yes)
+			)

Commit message: Made last changes to CAD, PCB, & journal. Ready for submission
Parts:
- K1, K2, K3, K4, K5, K6: footprint Relay_SMD:Relay_DPDT_Omron_G6K-2F -> Relay_SMD:Relay_DPDT_Omron_G6K-2F-Y
Changed lines of the file:
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@@
 			)
 		)
-		(property "Footprint" "Relay_SMD:Relay_DPDT_Omron_G6K-2F"
+		(property "Footprint" "Relay_SMD:Relay_DPDT_Omron_G6K-2F-Y"
 			(at 138.43 45.72 0)
 			(effects
@@
 			)
 		)
-		(property "Footprint" "Relay_SMD:Relay_DPDT_Omron_G6K-2F"
+		(property "Footprint" "Relay_SMD:Relay_DPDT_Omron_G6K-2F-Y"
 			(at 226.06 45.72 0)
 			(effects
@@
 			)
 		)
-		(property "Footprint" "Relay_SMD:Relay_DPDT_Omron_G6K-2F"
+		(property "Footprint" "Relay_SMD:Relay_DPDT_Omron_G6K-2F-Y"
 			(at 226.06 81.28 0)
 			(effects
@@
 			)
 		)
-		(property "Footprint" "Relay_SMD:Relay_DPDT_Omron_G6K-2F"
+		(property "Footprint" "Relay_SMD:Relay_DPDT_Omron_G6K-2F-Y"
 			(at 97.79 45.72 0)
 			(effects
@@
 			)
 		)
-		(property "Footprint" "Relay_SMD:Relay_DPDT_Omron_G6K-2F"
+		(property "Footprint" "Relay_SMD:Relay_DPDT_Omron_G6K-2F-Y"
 			(at 179.07 45.72 0)
 			(effects
@@
 			)
 		)
-		(property "Footprint" "Relay_SMD:Relay_DPDT_Omron_G6K-2F"
+		(property "Footprint" "Relay_SMD:Relay_DPDT_Omron_G6K-2F-Y"
 			(at 274.32 45.72 0)
 			(effects
